Commit message: Added axes permutation to align model with sensors.

File: diver_net/data/models/xacro/diver_model_unpermuted.xacro (robot description, xacro)
@@ -67,48 +67,48 @@
 	</xacro:OldJoint> -->
 	<xacro:OldJoint node="lower_back" parent="local">
-		<origin xyz="0 0 0" rpy="0 0 0" />
+		<origin xyz="0.1 0 -0.15" rpy="0 -1.57 0" />
     <box size="0.1 0.2 0.05"/>
     <color rgba="1 0 0 1" />
-    <origin xyz="0 0 0"/>
+    <origin xyz="0 0 0.3"/>
 	</xacro:OldJoint>
 	<xacro:Joint3d node="upper_body" parent="lower_back">
-    <origin xyz="0 0 0.35" rpy="0 0 0" />
+    <origin xyz="0 0 -0.15" rpy="3.14 -1.57 0" />
 		<mesh filename="package://diver_net/data/models/dae/torso.dae" />
-		<origin xyz="0 0 0" />
+		<origin xyz="0.35 0 -0.3" />
 	</xacro:Joint3d>
 	<xacro:Joint3d node="head" parent="upper_body">
-		<origin xyz="0.05 0 0.1" rpy="0 0 0" />
+		<origin xyz="0.1 0 0.1" rpy="0 0 0" />
     <mesh filename="package://diver_net/data/models/dae/head.dae" />
-		<origin xyz="0 0 0.5" />
+		<origin xyz="0.15 0 -0.15" />
 	</xacro:Joint3d>
 	<xacro:Joint3d node="left_thigh" parent="lower_back">
-    <origin xyz="0 0 0" rpy="0 0 0"/>
+    <origin xyz="-0.1 0 0" rpy="0 -1.57 0"/>
 		<mesh filename="package://diver_net/data/models/dae/left_thigh.dae" />
-    <origin xyz="0 0.1 0" />
+    <origin xyz="-0.05 0.08 -0.15" />
 	</xacro:Joint3d>
 	<xacro:Joint3d node="right_thigh" parent="lower_back">
-		<origin xyz="0 0 0" rpy="0 0 0"/>
+		<origin xyz="-0.1 0 0" rpy="0 -1.57 0"/>
     <mesh filename="package://diver_net/data/models/dae/right_thigh.dae" />
-		<origin xyz="0 -0.1 0" />
+		<origin xyz="-0.05 -0.08 -0.15" />
 	</xacro:Joint3d>
 	<xacro:Joint3d node="right_calf" parent="right_thigh">
-		<origin xyz="0 0 0" rpy="0 0 0"/>
+		<origin xyz="0 0 0" rpy="0 -1.57 0"/>
 		<mesh filename="package://diver_net/data/models/dae/right_leg.dae" />
-		<origin xyz="0 0 -0.4" />
+		<origin xyz="0.3 0 0" />
 	</xacro:Joint3d>
 	<xacro:Joint3d node="left_calf" parent="left_thigh">
-		<origin xyz="0 0 0" rpy="0 0 0"/>
+		<origin xyz="0 0 0" rpy="0 -1.57 0"/>
 		<mesh filename="package://diver_net/data/models/dae/left_leg.dae" />
-		<origin xyz="0 0 -0.4" />
+		<origin xyz="0.3 0 0" />
 	</xacro:Joint3d>
 	<xacro:Joint3d node="right_foot" parent="right_calf">
 		<origin xyz="0 0 0" rpy="0 0 0"/>
 		<mesh filename="package://diver_net/data/models/dae/right_flipper.dae" />
-    <origin xyz="0 0 -0.45" />
+    <origin xyz="0.42 0 0" />
 	</xacro:Joint3d>
 	<xacro:Joint3d node="left_foot" parent="left_calf">
 		<origin xyz="0 0 0" rpy="0 0 0"/>
 		<mesh filename="package://diver_net/data/models/dae/left_flipper.dae" />
-    <origin xyz="0 0 -0.45" />
+    <origin xyz="0.42 0 0" />
 	</xacro:Joint3d>
 	<xacro:OldJoint node="left_shoulder" parent="upper_body">
@@ -116,5 +116,5 @@
 		<box size="0.1 0.1 0.1" />
 		<color rgba="0 1 1 1" />
-		<origin xyz="0 0.15 0.5" />
+		<origin xyz="0.15 -0.15 -0.1" />
 	</xacro:OldJoint>
 		<xacro:OldJoint node="right_shoulder" parent="upper_body">
@@ -122,25 +122,25 @@
 		<box size="0.1 0.1 0.1" />
 		<color rgba="0 1 0 1" />
-	  <origin xyz="0 -0.15 0.5" />
+	  <origin xyz="0.15 0.15 -0.1" />
   </xacro:OldJoint>
 	<xacro:Joint3d node="left_upper_arm" parent="upper_body">
 		<origin xyz="0 0 0" rpy="0 0 -1.57"/>
 		<mesh filename="package://diver_net/data/models/dae/left_biceps.dae" />
-	  <origin xyz="0 0.2 0.5" />
+	  <origin xyz="0.15 -0.2 -0.1" />
   </xacro:Joint3d>
 	<xacro:Joint3d node="right_upper_arm" parent="upper_body">
 		<origin xyz="0 0 0" rpy="0 0 1.57"/>
 		<mesh filename="package://diver_net/data/models/dae/right_biceps.dae" />
-	  <origin xyz="0 -0.2 0.5" />
+	  <origin xyz="0.15 0.2 -0.1" />
   </xacro:Joint3d>
 	<xacro:Joint3d node="left_forearm" parent="left_upper_arm">
 		<origin xyz="0 0 0" rpy="0 0 -1.57"/>
 		<mesh filename="package://diver_net/data/models/dae/left_forearm.dae" />
-	  <origin xyz="0.3 0 0" />
+	  <origin xyz="0.25 0 0" />
   </xacro:Joint3d>
 	<xacro:Joint3d node="right_forearm" parent="right_upper_arm">
 		<origin xyz="0 0 0" rpy="0 0 1.57"/>
 		<mesh filename="package://diver_net/data/models/dae/right_forearm.dae" />
-	  <origin xyz="0.3 0 0" />
+	  <origin xyz="0.25 0 0" />
 	</xacro:Joint3d>
 	<xacro:Joint3d node="left_hand" parent="left_forearm">
@@ -152,5 +152,5 @@
 		<origin xyz="0 0 0" rpy="0 1.57 1.57"/>
 		<mesh filename="package://diver_net/data/models/dae/right_hand.dae" />
-		<origin xyz="0.25 0 0" />`
+		<origin xyz="0.25 0 0" />
 	</xacro:Joint3d>
 </robot>
