Commit message: Minor changes to diver model body parts positions

File: diver_net/data/models/xacro/diver_model.xacro (robot description, xacro)
@@ -68,40 +68,40 @@
 	<xacro:Joint3d node="upper_body" parent="lower_back">
     <origin xyz="0 0 -0.15" rpy="3.14 -1.57 0" />
-		<mesh filename="package://diver_model/models/torso.dae" />
+		<mesh filename="package://diver_net/data/models/dae/torso.dae" />
 		<origin xyz="0.35 0 -0.3" />
 	</xacro:Joint3d>
 	<xacro:Joint3d node="head" parent="upper_body">
-		<origin xyz="0 0 0.1" rpy="0 0 0" />
-    <mesh filename="package://diver_model/models/head.dae" />
+		<origin xyz="0.1 0 0.1" rpy="0 0 0" />
+    <mesh filename="package://diver_net/data/models/dae/head.dae" />
 		<origin xyz="0.15 0 -0.15" />
 	</xacro:Joint3d>
 	<xacro:Joint3d node="left_thigh" parent="lower_back">
     <origin xyz="-0.1 0 0" rpy="0 -1.57 0"/>
-		<mesh filename="package://diver_model/models/left_thigh.dae" />
+		<mesh filename="package://diver_net/data/models/dae/left_thigh.dae" />
     <origin xyz="-0.05 0.12 -0.15" />
 	</xacro:Joint3d>
 	<xacro:Joint3d node="right_thigh" parent="lower_back">
 		<origin xyz="-0.1 0 0" rpy="0 -1.57 0"/>
-    <mesh filename="package://diver_model/models/right_thigh.dae" />
+    <mesh filename="package://diver_net/data/models/dae/right_thigh.dae" />
 		<origin xyz="-0.05 -0.12 -0.15" />
 	</xacro:Joint3d>
 	<xacro:Joint3d node="right_calf" parent="right_thigh">
 		<origin xyz="0 0 0" rpy="0 -1.57 0"/>
-		<mesh filename="package://diver_model/models/right_leg.dae" />
+		<mesh filename="package://diver_net/data/models/dae/right_leg.dae" />
 		<origin xyz="0.3 0 0" />
 	</xacro:Joint3d>
 	<xacro:Joint3d node="left_calf" parent="left_thigh">
 		<origin xyz="0 0 0" rpy="0 -1.57 0"/>
-		<mesh filename="package://diver_model/models/left_leg.dae" />
+		<mesh filename="package://diver_net/data/models/dae/left_leg.dae" />
 		<origin xyz="0.3 0 0" />
 	</xacro:Joint3d>
 	<xacro:Joint3d node="right_foot" parent="right_calf">
 		<origin xyz="-0.03 0 0" rpy="0 0 0"/>
-		<mesh filename="package://diver_model/models/right_flipper.dae" />
+		<mesh filename="package://diver_net/data/models/dae/right_flipper.dae" />
     <origin xyz="0.47 0 0" />
 	</xacro:Joint3d>
 	<xacro:Joint3d node="left_foot" parent="left_calf">
 		<origin xyz="-0.03 0 0" rpy="0 0 0"/>
-		<mesh filename="package://diver_model/models/left_flipper.dae" />
+		<mesh filename="package://diver_net/data/models/dae/left_flipper.dae" />
     <origin xyz="0.47 0 0" />
 	</xacro:Joint3d>
@@ -110,5 +110,5 @@
 		<box size="0.1 0.1 0.1" />
 		<color rgba="0 1 1 1" />
-		<origin xyz="0.15 -0.15 -0.1" />
+		<origin xyz="0.15 -0.15 -0.15" />
 	</xacro:OldJoint>
 		<xacro:OldJoint node="right_shoulder" parent="upper_body">
@@ -116,34 +116,34 @@
 		<box size="0.1 0.1 0.1" />
 		<color rgba="0 1 0 1" />
-	  <origin xyz="0.15 0.15 -0.1" />
+	  <origin xyz="0.15 0.15 -0.15" />
   </xacro:OldJoint>
 	<xacro:Joint3d node="left_upper_arm" parent="left_shoulder">
 		<origin xyz="0 0 0" rpy="0 0 -1.57"/>
-		<mesh filename="package://diver_model/models/left_biceps.dae" />
-	  <origin xyz="0.05 0 -0.05" />
+		<mesh filename="package://diver_net/data/models/dae/left_biceps.dae" />
+	  <origin xyz="0.05 0 0.0" />
   </xacro:Joint3d>
 	<xacro:Joint3d node="right_upper_arm" parent="right_shoulder">
 		<origin xyz="0 0 0" rpy="0 0 1.57"/>
-		<mesh filename="package://diver_model/models/right_biceps.dae" />
-	  <origin xyz="0.05 0 -0.05" />
+		<mesh filename="package://diver_net/data/models/dae/right_biceps.dae" />
+	  <origin xyz="0.05 0 0.0" />
   </xacro:Joint3d>
 	<xacro:Joint3d node="left_forearm" parent="left_upper_arm">
 		<origin xyz="0 0 0" rpy="0 0 -1.57"/>
-		<mesh filename="package://diver_model/models/left_forearm.dae" />
+		<mesh filename="package://diver_net/data/models/dae/left_forearm.dae" />
 	  <origin xyz="0.25 0 0" />
   </xacro:Joint3d>
 	<xacro:Joint3d node="right_forearm" parent="right_upper_arm">
 		<origin xyz="0 0 0" rpy="0 0 1.57"/>
-		<mesh filename="package://diver_model/models/right_forearm.dae" />
+		<mesh filename="package://diver_net/data/models/dae/right_forearm.dae" />
 	  <origin xyz="0.25 0 0" />
 	</xacro:Joint3d>
 	<xacro:Joint3d node="left_hand" parent="left_forearm">
 		<origin xyz="0 0 0" rpy="0 0 -1.57"/>
-		<mesh filename="package://diver_model/models/left_hand.dae" />
+		<mesh filename="package://diver_net/data/models/dae/left_hand.dae" />
 		<origin xyz="0.25 0 0" />
 	</xacro:Joint3d>
 	<xacro:Joint3d node="right_hand" parent="right_forearm">
 		<origin xyz="0 0 0" rpy="0 0 1.57"/>
-		<mesh filename="package://diver_model/models/right_hand.dae" />
+		<mesh filename="package://diver_net/data/models/dae/right_hand.dae" />
 		<origin xyz="0.25 0 0" />
 	</xacro:Joint3d>

Commit message: Added calibration/initialization

File: diver_net/data/models/xacro/diver_model.xacro (robot description, xacro)
@@ -60,4 +60,10 @@
 		</joint>
 	</xacro:macro>
+	<!-- <xacro:OldJoint node="lower_back" parent="local">
+		<origin xyz="0 0 0" rpy="0 0 0" />
+    <box size="0.1 0.2 0.05"/>
+    <color rgba="1 0 0 1" />
+    <origin xyz="0 0 0"/>
+	</xacro:OldJoint> -->
 	<xacro:OldJoint node="lower_back" parent="local">
 		<origin xyz="0.1 0 -0.15" rpy="0 -1.57 0" />

Commit message: Updates to the diver net models.

File: diver_net/data/models/xacro/diver_model.xacro (robot description, xacro)
@@ -152,5 +152,5 @@
 		<origin xyz="0 0 0" rpy="0 1.57 1.57"/>
 		<mesh filename="package://diver_net/data/models/dae/right_hand.dae" />
-		<origin xyz="0.25 0 0" />`
+		<origin xyz="0.25 0 0" />
 	</xacro:Joint3d>
 </robot>

File: diver_net/data/models/xacro/diver_model_base.xacro (robot description, xacro)
@@ -2,4 +2,5 @@
 <robot xmlns:xacro="http://www.ros.org/wiki/xacro" name="diver">
 	<link name="local" />
+	<xacro:property name="pi" value="3.1415926535897931" />
 	<xacro:macro name="Joint3d"
 		params="node parent *origin *geometry *origin_joint">
@@ -67,48 +68,48 @@
 	</xacro:OldJoint> -->
 	<xacro:OldJoint node="lower_back" parent="local">
-		<origin xyz="0.1 0 -0.15" rpy="0 -1.57 0" />
+		<origin xyz="0 0 0" rpy="0 0 0" />
     <box size="0.1 0.2 0.05"/>
     <color rgba="1 0 0 1" />
-    <origin xyz="0 0 0.3"/>
+    <origin xyz="0 0 0"/>
 	</xacro:OldJoint>
 	<xacro:Joint3d node="upper_body" parent="lower_back">
-    <origin xyz="0 0 -0.15" rpy="3.14 -1.57 0" />
+    <origin xyz="0 0 0.35" rpy="0 0 0" />
 		<mesh filename="${mesh_path}torso.${mesh_extension}" />
-		<origin xyz="0.35 0 -0.3" />
+		<origin xyz="0 0 0" />
 	</xacro:Joint3d>
 	<xacro:Joint3d node="head" parent="upper_body">
-		<origin xyz="0.1 0 0.1" rpy="0 0 0" />
+		<origin xyz="0.05 0 0.1" rpy="0 0 0" />
     <mesh filename="${mesh_path}head.${mesh_extension}" />
-		<origin xyz="0.15 0 -0.15" />
+		<origin xyz="0 0 0.5" />
 	</xacro:Joint3d>
 	<xacro:Joint3d node="left_thigh" parent="lower_back">
-    <origin xyz="-0.1 0 0" rpy="0 -1.57 0"/>
+    <origin xyz="0 0 0" rpy="0 0 0"/>
 		<mesh filename="${mesh_path}left_thigh.${mesh_extension}" />
-    <origin xyz="-0.05 0.08 -0.15" />
+    <origin xyz="0 0.1 0" />
 	</xacro:Joint3d>
 	<xacro:Joint3d node="right_thigh" parent="lower_back">
-		<origin xyz="-0.1 0 0" rpy="0 -1.57 0"/>
+		<origin xyz="0 0 0" rpy="0 0 0"/>
     <mesh filename="${mesh_path}right_thigh.${mesh_extension}" />
-		<origin xyz="-0.05 -0.08 -0.15" />
+		<origin xyz="0 -0.1 0" />
 	</xacro:Joint3d>
 	<xacro:Joint3d node="right_calf" parent="right_thigh">
-		<origin xyz="0 0 0" rpy="0 -1.57 0"/>
+		<origin xyz="0 0 0" rpy="0 0 0"/>
 		<mesh filename="${mesh_path}right_leg.${mesh_extension}" />
-		<origin xyz="0.3 0 0" />
+		<origin xyz="0 0 -0.4" />
 	</xacro:Joint3d>
 	<xacro:Joint3d node="left_calf" parent="left_thigh">
-		<origin xyz="0 0 0" rpy="0 -1.57 0"/>
+		<origin xyz="0 0 0" rpy="0 0 0"/>
 		<mesh filename="${mesh_path}left_leg.${mesh_extension}" />
-		<origin xyz="0.3 0 0" />
+		<origin xyz="0 0 -0.4" />
 	</xacro:Joint3d>
 	<xacro:Joint3d node="right_foot" parent="right_calf">
 		<origin xyz="0 0 0" rpy="0 0 0"/>
 		<mesh filename="${mesh_path}right_flipper.${mesh_extension}" />
-    <origin xyz="0.42 0 0" />
+    <origin xyz="0 0 -0.45" />
 	</xacro:Joint3d>
 	<xacro:Joint3d node="left_foot" parent="left_calf">
 		<origin xyz="0 0 0" rpy="0 0 0"/>
 		<mesh filename="${mesh_path}left_flipper.${mesh_extension}" />
-    <origin xyz="0.42 0 0" />
+    <origin xyz="0 0 -0.45" />
 	</xacro:Joint3d>
 	<xacro:OldJoint node="left_shoulder" parent="upper_body">
@@ -116,5 +117,5 @@
 		<box size="0.1 0.1 0.1" />
 		<color rgba="0 1 1 1" />
-		<origin xyz="0.15 -0.15 -0.1" />
+		<origin xyz="0 0.15 0.5" />
 	</xacro:OldJoint>
 		<xacro:OldJoint node="right_shoulder" parent="upper_body">
@@ -122,33 +123,33 @@
 		<box size="0.1 0.1 0.1" />
 		<color rgba="0 1 0 1" />
-	  <origin xyz="0.15 0.15 -0.1" />
+	  <origin xyz="0 -0.15 0.5" />
   </xacro:OldJoint>
 	<xacro:Joint3d node="left_upper_arm" parent="upper_body">
-		<origin xyz="0 0 0" rpy="0 0 -1.57"/>
+		<origin xyz="0 0 0" rpy="0 0 -${0.5 * pi}"/>
 		<mesh filename="${mesh_path}left_biceps.${mesh_extension}" />
-	  <origin xyz="0.15 -0.2 -0.1" />
+	  <origin xyz="0 0.2 0.5" />
   </xacro:Joint3d>
 	<xacro:Joint3d node="right_upper_arm" parent="upper_body">
-		<origin xyz="0 0 0" rpy="0 0 1.57"/>
+		<origin xyz="0 0 0" rpy="0 0 ${0.5 * pi}"/>
 		<mesh filename="${mesh_path}right_biceps.${mesh_extension}" />
-	  <origin xyz="0.15 0.2 -0.1" />
+	  <origin xyz="0 -0.2 0.5" />
   </xacro:Joint3d>
 	<xacro:Joint3d node="left_forearm" parent="left_upper_arm">
-		<origin xyz="0 0 0" rpy="0 0 -1.57"/>
+		<origin xyz="0 0 0" rpy="0 0 -${0.5 * pi}"/>
 		<mesh filename="${mesh_path}left_forearm.${mesh_extension}" />
-	  <origin xyz="0.25 0 0" />
+	  <origin xyz="0.3 0 0" />
   </xacro:Joint3d>
 	<xacro:Joint3d node="right_forearm" parent="right_upper_arm">
-		<origin xyz="0 0 0" rpy="0 0 1.57"/>
+		<origin xyz="0 0 0" rpy="0 0 ${0.5 * pi}"/>
 		<mesh filename="${mesh_path}right_forearm.${mesh_extension}" />
-	  <origin xyz="0.25 0 0" />
+	  <origin xyz="0.3 0 0" />
 	</xacro:Joint3d>
 	<xacro:Joint3d node="left_hand" parent="left_forearm">
-		<origin xyz="0 0 0" rpy="0 1.57 -1.57"/>
+		<origin xyz="0 0 0" rpy="0 ${0.5 * pi} -${0.5 * pi}"/>
 		<mesh filename="${mesh_path}left_hand.${mesh_extension}" />
 		<origin xyz="0.25 0 0" />
 	</xacro:Joint3d>
 	<xacro:Joint3d node="right_hand" parent="right_forearm">
-		<origin xyz="0 0 0" rpy="0 1.57 1.57"/>
+		<origin xyz="0 0 0" rpy="0 ${0.5 * pi} ${0.5 * pi}"/>
 		<mesh filename="${mesh_path}right_hand.${mesh_extension}" />
 		<origin xyz="0.25 0 0" />

File: diver_net/data/models/xacro/uwsim_diver_model.urdf.xacro (robot description, xacro)
@@ -1,5 +1,5 @@
 <?xml version="1.0"?>
 <robot xmlns:xacro="http://www.ros.org/wiki/xacro" name="diver">
- 	<xacro:property name="mesh_path" value="models/osgt/" />
+ 	<xacro:property name="mesh_path" value="mesh/osgt/" />
  	<xacro:property name="mesh_extension" value="osgt" />
  	<xacro:include filename="$(find diver_net)/data/models/xacro/diver_model_base.xacro" />
