Commit message: Added divernet gui in launch file, and preparation for pose calibration with gui, + forgotten setup.py from previous commit.

File: diver_net/data/models/xacro/diver_model_pose_calibration.xacro (robot description, xacro)
@@ -1,5 +1,5 @@
 <?xml version="1.0"?>
-<robot xmlns:xacro="http://www.ros.org/wiki/xacro" name="diver">
-	<link name="local" />
+<robot xmlns:xacro="http://www.ros.org/wiki/xacro" name="diver2">
+  <link name="local" />
 	<xacro:macro name="Joint3d"
 		params="node parent *origin *geometry *origin_joint">
@@ -60,5 +60,5 @@
 		</joint>
 	</xacro:macro>
-	<!-- <xacro:OldJoint node="lower_back" parent="local">
+	<!-- <xacro:OldJoint node="pose_calibration/lower_back" parent="pose_calibration/local">
 		<origin xyz="0 0 0" rpy="0 0 0" />
     <box size="0.1 0.2 0.05"/>
@@ -66,5 +66,5 @@
     <origin xyz="0 0 0"/>
 	</xacro:OldJoint> -->
-	<xacro:OldJoint node="lower_back" parent="local">
+  <xacro:OldJoint node="pose_calibration/lower_back" parent="local">
 		<origin xyz="0 0 0" rpy="0 0 0" />
     <box size="0.1 0.2 0.05"/>
@@ -72,45 +72,45 @@
     <origin xyz="0 0 0"/>
 	</xacro:OldJoint>
-	<xacro:Joint3d node="upper_body" parent="lower_back">
+	<xacro:Joint3d node="pose_calibration/upper_body" parent="pose_calibration/lower_back">
     <origin xyz="0 0 0.35" rpy="0 0 0" />
 		<mesh filename="package://diver_net/data/mesh/dae/torso.dae" />
 		<origin xyz="0 0 0" />
 	</xacro:Joint3d>
-	<xacro:Joint3d node="head" parent="upper_body">
+	<xacro:Joint3d node="pose_calibration/head" parent="pose_calibration/upper_body">
 		<origin xyz="0.05 0 0.1" rpy="0 0 0" />
     <mesh filename="package://diver_net/data/mesh/dae/head.dae" />
 		<origin xyz="0 0 0.5" />
 	</xacro:Joint3d>
-	<xacro:Joint3d node="left_thigh" parent="lower_back">
+	<xacro:Joint3d node="pose_calibration/left_thigh" parent="pose_calibration/lower_back">
     <origin xyz="0 0 0" rpy="0 0 0"/>
 		<mesh filename="package://diver_net/data/mesh/dae/left_thigh.dae" />
     <origin xyz="0 0.1 0" />
 	</xacro:Joint3d>
-	<xacro:Joint3d node="right_thigh" parent="lower_back">
+	<xacro:Joint3d node="pose_calibration/right_thigh" parent="pose_calibration/lower_back">
 		<origin xyz="0 0 0" rpy="0 0 0"/>
     <mesh filename="package://diver_net/data/mesh/dae/right_thigh.dae" />
 		<origin xyz="0 -0.1 0" />
 	</xacro:Joint3d>
-	<xacro:Joint3d node="right_calf" parent="right_thigh">
+	<xacro:Joint3d node="pose_calibration/right_calf" parent="pose_calibration/right_thigh">
 		<origin xyz="0 0 0" rpy="0 0 0"/>
 		<mesh filename="package://diver_net/data/mesh/dae/right_leg.dae" />
 		<origin xyz="0 0 -0.4" />
 	</xacro:Joint3d>
-	<xacro:Joint3d node="left_calf" parent="left_thigh">
+	<xacro:Joint3d node="pose_calibration/left_calf" parent="pose_calibration/left_thigh">
 		<origin xyz="0 0 0" rpy="0 0 0"/>
 		<mesh filename="package://diver_net/data/mesh/dae/left_leg.dae" />
 		<origin xyz="0 0 -0.4" />
 	</xacro:Joint3d>
-	<xacro:Joint3d node="right_foot" parent="right_calf">
+	<xacro:Joint3d node="pose_calibration/right_foot" parent="pose_calibration/right_calf">
 		<origin xyz="0 0 0" rpy="0 0 0"/>
 		<mesh filename="package://diver_net/data/mesh/dae/right_flipper.dae" />
     <origin xyz="0 0 -0.45" />
 	</xacro:Joint3d>
-	<xacro:Joint3d node="left_foot" parent="left_calf">
+	<xacro:Joint3d node="pose_calibration/left_foot" parent="pose_calibration/left_calf">
 		<origin xyz="0 0 0" rpy="0 0 0"/>
 		<mesh filename="package://diver_net/data/mesh/dae/left_flipper.dae" />
     <origin xyz="0 0 -0.45" />
 	</xacro:Joint3d>
-	<xacro:OldJoint node="left_shoulder" parent="upper_body">
+	<xacro:OldJoint node="pose_calibration/left_shoulder" parent="pose_calibration/upper_body">
 		<origin xyz="0 0 0" rpy="0 0 0"/>
 		<box size="0.1 0.1 0.1" />
@@ -118,5 +118,5 @@
 		<origin xyz="0 0.15 0.5" />
 	</xacro:OldJoint>
-		<xacro:OldJoint node="right_shoulder" parent="upper_body">
+		<xacro:OldJoint node="pose_calibration/right_shoulder" parent="pose_calibration/upper_body">
 		<origin xyz="0 0 0" rpy="0 0 0"/>
 		<box size="0.1 0.1 0.1" />
@@ -124,30 +124,30 @@
 	  <origin xyz="0 -0.15 0.5" />
   </xacro:OldJoint>
-	<xacro:Joint3d node="left_upper_arm" parent="upper_body">
+	<xacro:Joint3d node="pose_calibration/left_upper_arm" parent="pose_calibration/upper_body">
 		<origin xyz="0 0 0" rpy="0 0 -1.57"/>
 		<mesh filename="package://diver_net/data/mesh/dae/left_biceps.dae" />
 	  <origin xyz="0 0.2 0.5" />
   </xacro:Joint3d>
-	<xacro:Joint3d node="right_upper_arm" parent="upper_body">
+	<xacro:Joint3d node="pose_calibration/right_upper_arm" parent="pose_calibration/upper_body">
 		<origin xyz="0 0 0" rpy="0 0 1.57"/>
 		<mesh filename="package://diver_net/data/mesh/dae/right_biceps.dae" />
 	  <origin xyz="0 -0.2 0.5" />
   </xacro:Joint3d>
-	<xacro:Joint3d node="left_forearm" parent="left_upper_arm">
+	<xacro:Joint3d node="pose_calibration/left_forearm" parent="pose_calibration/left_upper_arm">
 		<origin xyz="0 0 0" rpy="0 0 -1.57"/>
 		<mesh filename="package://diver_net/data/mesh/dae/left_forearm.dae" />
 	  <origin xyz="0.3 0 0" />
   </xacro:Joint3d>
-	<xacro:Joint3d node="right_forearm" parent="right_upper_arm">
+	<xacro:Joint3d node="pose_calibration/right_forearm" parent="pose_calibration/right_upper_arm">
 		<origin xyz="0 0 0" rpy="0 0 1.57"/>
 		<mesh filename="package://diver_net/data/mesh/dae/right_forearm.dae" />
 	  <origin xyz="0.3 0 0" />
 	</xacro:Joint3d>
-	<xacro:Joint3d node="left_hand" parent="left_forearm">
+	<xacro:Joint3d node="pose_calibration/left_hand" parent="pose_calibration/left_forearm">
 		<origin xyz="0 0 0" rpy="0 1.57 -1.57"/>
 		<mesh filename="package://diver_net/data/mesh/dae/left_hand.dae" />
 		<origin xyz="0.25 0 0" />
 	</xacro:Joint3d>
-	<xacro:Joint3d node="right_hand" parent="right_forearm">
+	<xacro:Joint3d node="pose_calibration/right_hand" parent="pose_calibration/right_forearm">
 		<origin xyz="0 0 0" rpy="0 1.57 1.57"/>
 		<mesh filename="package://diver_net/data/mesh/dae/right_hand.dae" />
